File: POWER-rev-1/POWER-rev-1.kicad_pcb (KiCad board)
At the start: 2 copper layers, 85 parts, among them SW1 EG25-switch-CSS-1210MC, SW2 MIC-switch-CSS-1210MC, SW3 CAM-switch-CSS-1210MC, U1 BAT-CONNECTOR-FLTS22WR00, U2 MP3429GL-Z, U3 BQ25792RQMR, U4 22V-boost-AP3032KTR-G1, U5 TPS65023BRSBR

Commit message: replace 0ohm resistors with jumpers
Parts:
- added J1: PINHD_1x6_Female, SL_Connectors:PinHeader_1x06_P2.54mm_Vertical, F.Cu at (169.3, 83.3)
- added J2: PINHD_1x6_Female, SL_Connectors:PinHeader_1x06_P2.54mm_Vertical, F.Cu at (187.1, 84.9)
- added R15: 10Ω, SPIRIT-footprints:0805-resistor, F.Cu at (176.2, 107.6)
- added R30: 0Ω, SPIRIT-footprints:0805-resistor, F.Cu at (171.0, 63.5)
- added R31: 0Ω, SPIRIT-footprints:0805-resistor, F.Cu at (171.0, 66.3)
- added R32: 0Ω, SPIRIT-footprints:0805-resistor, F.Cu at (171.0, 69.2)
