File: POWER-rev-1/POWER-rev-1.kicad_pcb (KiCad board)
At the start: 2 copper layers, 91 parts, among them J1 PINHD_1x6_Female, J2 PINHD_1x6_Female, SW1 EG25-switch-CSS-1210MC, SW2 MIC-switch-CSS-1210MC, SW3 CAM-switch-CSS-1210MC, U1 BAT-CONNECTOR-FLTS22WR00, U2 MP3429GL-Z, U3 BQ25792RQMR, U4 22V-boost-AP3032KTR-G1, U5 TPS65023BRSBR

Commit message: fix bad switch connections
Parts:
- added R15: 10Ω, SPIRIT-footprints:0805-resistor, F.Cu at (154.9, 118.0)
Connections:
- SW1 pad 2: EN3V3A SW OUT -> unconnected-(SW1-Pad2)
- SW1 pad 3: unconnected-(SW1-Pad3) -> EN3V3A SW OUT
- SW2 pad 2: MICSWITCH -> unconnected-(SW2-Pad2)
- SW2 pad 3: unconnected-(SW2-Pad3) -> MICSWITCH
- SW3 pad 2: Net-(Q2-G) -> unconnected-(SW3-Pad2)
- SW3 pad 3: unconnected-(SW3-Pad3) -> CAMSWITCH
Changed lines of the file:
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@@
 		(capping no)
 		(filling no)
-		(zone_defaults)
 		(pcbplotparams
 			(layerselection 0x00000000_00000000_55555555_5755f5ff)
@@
 			)
 		)
-		(property "Datasheet" "CSS-1210MC"
+		(property "Datasheet" "https://www.nidec-components.com/e/catalog/switch/css.pdf"
 			(at 0 0 0)
 			(layer "F.Fab")
@@
 			(layers "*.Cu" "*.Mask")
 			(remove_unused_layers no)
-			(net "EN3V3A SW OUT")
+			(net "unconnected-(SW1-Pad2)")
 			(pinfunction "2_2")
-			(pintype "unspecified")
+			(pintype "unspecified+no_connect")
 		)
 		(pad "3" thru_hole circle
@@
 			(layers "*.Cu" "*.Mask")
 			(remove_unused_layers no)
-			(net "unconnected-(SW1-Pad3)")
+			(net "EN3V3A SW OUT")
 			(pinfunction "3_3")
-			(pintype "unspecified+no_connect")
+			(pintype "unspecified")
 		)
 		(embedded_fonts no)
@@
 			(layers "*.Cu" "*.Mask")
 			(remove_unused_layers no)
-			(net "Net-(Q2-G)")
+			(net "unconnected-(SW3-Pad2)")
 			(pinfunction "2_2")
-			(pintype "unspecified")
+			(pintype "unspecified+no_connect")
 		)
 		(pad "3" thru_hole circle
@@
 			(layers "*.Cu" "*.Mask")
 			(remove_unused_layers no)
-			(net "unconnected-(SW3-Pad3)")
+			(net "CAMSWITCH")
 			(pinfunction "3_3")
-			(pintype "unspecified+no_connect")
+			(pintype "unspecified")
 		)
 		(embedded_fonts no)
@@
 		)
 	)
+	(footprint "SPIRIT-footprints:0805-resistor"
+		(layer "F.Cu")
+		(at 154.875 118.05)
+		(property "Reference" "R15"
+			(at -0.2 -1.3 0)
+			(layer "F.SilkS")
+			(effects
+				(font
+					(size 0.64 0.64)
+					(thickness 0.15)
+				)
+			)
+		)
+		(property "Value" "10Ω"
+			(at 1.8 0 0)
+			(layer "F.Fab")
+			(effects
+				(font
+					(size 0.64 0.64)
+					(thickness 0.15)
+				)
+			)
+		)
+		(property "Datasheet" ""
+			(at 0 0 0)
+			(layer "F.Fab")
+			(hide yes)
+			(effects
+				(font
+					(size 1.27 1.27)
+					(thickness 0.15)
+				)
+			)
+		)
+		(property "Description" "Resistor"
+			(at 0 0 0)
+			(layer "F.Fab")
+			(hide yes)
+			(effects
+				(font
+					(size 1.27 1.27)
+					(thickness 0.15)
+				)
+			)
+		)
+		(property "MPN" "RC0805FR-0710RL"
+			(at 0 0 0)
+			(unlocked yes)
+			(layer "F.Fab")
+			(hide yes)
+			(effects
+				(font
+					(size 1 1)
+					(thickness 0.15)
+				)
+			)
+		)
+		(property ki_fp_filters "R_*")
+		(sheetname "/")
+		(sheetfile "POWER-rev-1.kicad_sch")
+		(units
+			(unit
+				(name "A")
+				(pins "1" "2")
+			)
+		)
+		(attr smd)
+		(duplicate_pad_numbers_are_jumpers no)
+		(fp_line
+			(start -0.2 -0.4)
+			(end 0.2 -0.4)
+			(stroke
+				(width 0.127)
+				(type solid)
+			)
+			(layer "F.SilkS")
+		)
+		(fp_line
+			(start -0.2 0.4)
+			(end -0.2 -0.4)
+			(stroke
+				(width 0.127)
+				(type solid)
+			)
+			(layer "F.SilkS")
+		)
+		(fp_line
+			(start -0.2 0.4)
+			(end 0.2 0.4)
+			(stroke
+				(width 0.127)
+				(type solid)
+			)
+			(layer "F.SilkS")
+		)
+		(fp_line
+			(start 0 -0.4)
+			(end 0 -0.6)
+			(stroke
+				(width 0.127)
+				(type solid)
+			)
+			(layer "F.SilkS")
+		)
+		(fp_line
+			(start 0 0.6)
+			(end 0 0.4)
+			(stroke
+				(width 0.127)
+				(type solid)
+			)
+			(layer "F.SilkS")
+		)
+		(fp_line
+			(start 0.2 0.4)
+			(end 0.2 -0.4)
+			(stroke
+				(width 0.127)
+				(type solid)
+			)
+			(layer "F.SilkS")
+		)
+		(fp_line
+			(start -1.5 -0.875)
+			(end -1.5 0.875)
+			(stroke
+				(width 0.05)
+				(type solid)
+			)
+			(layer "F.CrtYd")
+		)
+		(fp_line
+			(start -1.5 0.875)
+			(end 1.5 0.875)
+			(stroke
+				(width 0.05)
+				(type solid)
+			)
+			(layer "F.CrtYd")
+		)
+		(fp_line
+			(start 1.5 -0.875)
+			(end -1.5 -0.875)
+			(stroke
+				(width 0.05)
+				(type solid)
+			)
+			(layer "F.CrtYd")
+		)
+		(fp_line
+			(start 1.5 0.875)
+			(end 1.5 -0.875)
+			(stroke
+				(width 0.05)
+				(type solid)
+			)
+			(layer "F.CrtYd")
+		)
+		(fp_line
+			(start -1 -0.625)
+			(end -1 0.625)
+			(stroke
+				(width 0.127)
+				(type solid)
+			)
+			(layer "F.Fab")
+		)
+		(fp_line
+			(start -1 -0.625)
+			(end 1 -0.625)
+			(stroke
+				(width 0.127)
+				(type solid)
+			)
+			(layer "F.Fab")
+		)
+		(fp_line
+			(start -1 0.625)
+			(end 1 0.625)
+			(stroke
+				(width 0.127)
+				(type solid)
+			)
+			(layer "F.Fab")
+		)
+		(fp_line
+			(start 1 -0.625)
+			(end 1 0.625)
+			(stroke
+				(width 0.127)
+				(type solid)
+			)
+			(layer "F.Fab")
+		)
+		(pad "1" smd rect
+			(at -0.9 0)
+			(size 0.7 1.3)
+			(layers "F.Cu" "F.Mask" "F.Paste")
+			(net "SYS")
+			(pintype "passive")
+			(solder_mask_margin 0.102)
+		)
+		(pad "2" smd rect
+			(at 0.9 0)
+			(size 0.7 1.3)
+			(layers "F.Cu" "F.Mask" "F.Paste")
+			(net "Net-(U5-VCC)")
+			(pintype "passive")
+			(solder_mask_margin 0.102)
+		)
+		(embedded_fonts no)
+		(model "${KIPRJMOD}/component-libs/SPIRIT-3D-models/1K-05W-0805-RES_ERJP06J102V.step"
+			(offset
+				(xyz 0 0 0.5)
+			)
+			(scale
+				(xyz 1 1 1)
+			)
+			(rotate
+				(xyz 90 -0 -0)
+			)
+		)
+	)
 	(footprint "SPIRIT-footprints:0603-capacitor"
 		(layer "F.Cu")
@@
 			(layers "*.Cu" "*.Mask")
 			(remove_unused_layers no)
-			(net "MICSWITCH")
+			(net "unconnected-(SW2-Pad2)")
 			(pinfunction "2_2")
-			(pintype "unspecified")
+			(pintype "unspecified+no_connect")
 		)
 		(pad "3" thru_hole circle
@@
 			(layers "*.Cu" "*.Mask")
 			(remove_unused_layers no)
-			(net "unconnected-(SW2-Pad3)")
+			(net "MICSWITCH")
 			(pinfunction "3_3")
-			(pintype "unspecified+no_connect")
+			(pintype "unspecified")
 		)
 		(embedded_fonts no)
