File: POWER-rev-1/POWER-rev-1.kicad_sch (KiCad schematic)
At the start: 93 parts, among them SW1 EG25-switch-CSS-1210MC, SW2 MIC-switch-CSS-1210MC, SW3 CAM-switch-CSS-1210MC, U1 BAT-CONNECTOR-FLTS22WR00, U2 MP3429GL-Z, U3 BQ25792RQMR, U4 22V-boost-AP3032KTR-G1, U5 TPS65023BRSBR

Commit message: replace 0ohm resistors with jumpers
Parts:
- removed R17, R20, R24: 0Ω, SPIRIT-footprints:1K-05W-0805-RES_ERJP06J102V, symbol SPIRIT-components:1K-05W-0805-RES_ERJP06J102V
- removed R30, R31, R32: 0Ω, SPIRIT-footprints:0805-resistor, symbol SPIRIT-components:1K-05W-0805-RES_ERJP06J102V
- added J1, J2: PINHD_1x6_Female, SL_Connectors:PinHeader_1x06_P2.54mm_Vertical, symbol SL_Pin_Headers:PINHD_1x6_Female
- R15: footprint (none) -> SPIRIT-footprints:0805-resistor
Connections:
- net 1V8: now also J1.4
- net 3V3A: now also J1.2
- net 3V3B: now also J1.6
- net DEFDCDC1 DIVIDER: now also J1.1
- net SYS: now also J2.1, J2.3, J2.5
- net at C30.1, U5.6 (VINDCDC1): now also J2.2
- net at C44.1, L5.1, U5.2 (VDCDC3): now also J1.5
- net at C54.1, U5.5 (VINDCDC3): now also J2.6
- net at C53.1, U5.36 (VINDCDC2): now also J2.4
- net at C43.1, L4.1, U5.33 (VDCDC2): now also J1.3
Other:
- moved on the sheet: C29, C30, C36, C43, C44, C52, C53, C54, L4, L5, L6, R15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

Commit message: fix bad switch connections
Parts:
- removed Q1: (no value), SPIRIT-footprints:NMOS-BSC0902NSIATMA1-PG-TDSON-8-6-IC_ISC037N03L5ISATMA1, symbol SPIRIT-components:NMOS-BSC0902NSI
- removed Q2: (no value), SPIRIT-footprints:gpio-driver-transistor-fix-SOT65P210X110-3N, symbol SPIRIT-components:gpio-driver-transistor-BSS816NWH6327XTSA1
- removed R14: 1K-05W-0805, SPIRIT-footprints:1K-05W-0805-RES_ERJP06J102V, symbol SPIRIT-components:1K-05W-0805-RES_ERJP06J102V
- F1: MPN (none) -> 1210L900SLPR
Connections:
- net CAMSWITCH: now also SW3.3
- net EN3V3A SW OUT: now also SW1.3; no longer SW1.2
- net MICSWITCH: now also SW2.3; no longer SW2.2
Other:
- note added: "CAMSWITCH needs to go to the enable pin of the camera (CAM_IO0)"
- note added: "resettable fuse: I_{hold} = 9A I_{trip} = 18A time to trip = 2s"
- note removed: "TBD: Camera can be allowed to turn on, if this switch is put between cam gpio, and CM5 cam gpio as a valve. This way a reboot isnt needed to detect camera."
- note removed: "This FET can be used for the dual input application of the BQ25792 - see datasheet"
- note removed: "resettable fuse: I_{hold} = 9A I_{trip} = 18A"
